File: eval-boards/Eval-GP-Board/Second order filtering.sch (KiCad schematic (older format))
At the start: 13 parts, among them J8 TP5, J9 TP6, U3 ADA4807-1

Commit message: Updated schematic
均采用双运放，前级4522可以单运放工作也可以级联工作
Parts:
- removed C17: C, Capacitor_SMD:C_0603_1608Metric, symbol Device:C
- removed U3: ADA4807-1, Package_SO:SOIC-8_3.9x4.9mm_P1.27mm, symbol Amplifier_Operational:ADA4807-1
- added C19, C20: C, Capacitor_SMD:C_0603_1608Metric, symbol Device:C
- added J15: TP8, TestPoint:TestPoint_Pad_D2.0mm, symbol Connector:Conn_01x01_Male
- added J7: TP6, TestPoint:TestPoint_Pad_D2.0mm, symbol Connector:Conn_01x01_Male
- added R19, R25, R26, R27, R28, R29, R30: R, Resistor_SMD:R_0603_1608Metric, symbol Device:R
- added U3: ADA4807-2ARM, Package_SO:SOIC-8_3.9x4.9mm_P1.27mm, symbol Amplifier_Operational:ADA4807-2ARM
- J9: value TP6 -> TP7
Connections:
- net GND: now also C19.2, R19.1, R27.2
- net VCC: now also U3.8 (V+)
- net VEE: now also U3.4 (V-)
- net at C14.2, R10.1: now also U3.3 (+)
- net at R11.2: now also C15.1, R29.2, U3.1
- removed net OUT: C15.1, J9.1 (Pin_1), R11.1
- net signal_in renamed signal_in_A
- new net: R11.1, R19.2, U3.2 (-)
- new net: C19.1, R26.1, U3.5 (+)
- new net: R27.1, R28.2, U3.6 (-)
- new net: C20.1, R28.1, R30.2, U3.7
- new net: C20.2, R25.1, R26.2
- new net OUT_A: J9.1 (Pin_1), R29.1
- new net OUT_B: J15.1 (Pin_1), R30.1
- new net signal_in_B: J7.1 (Pin_1), R25.2
- no-connect marks 1 -> 0
Other:
- note removed: "R11 C17 to prevent oscillation\nC17 0.001u-0.1uF\nR11=R9+R10"
- moved on the sheet: C11, C12, C13, C14, C15, C16, J8, J9, R10, R11, R9
