File: eval-boards/HMC346AMS8GE/HMC346AMS8GE.kicad_pcb (KiCad board)
At the start: 2 copper layers, 8 parts, among them J1 Conn_Coaxial, J2 Conn_Coaxial, J3 Conn_01x04_Male, U1 HMC346AMS8GE

Commit message: final vision
最终版
Parts:
- added REF**: PinSocket_1x01_P1.27mm_Vertical, Connector_PinSocket_1.27mm:PinSocket_1x01_P1.27mm_Vertical, F.Cu at (121.9, 110.5)
- added REF**: PinSocket_1x01_P1.27mm_Vertical, Connector_PinSocket_1.27mm:PinSocket_1x01_P1.27mm_Vertical, F.Cu at (142.2, 110.5)
- added TP1: TestPoint_Pad_D2.0mm, TestPoint:TestPoint_Pad_D2.0mm, F.Cu at (124.5, 114.3)
- added TP2: TestPoint_Pad_D2.0mm, TestPoint:TestPoint_Pad_D2.0mm, F.Cu at (140.3, 114.3)
- GND V2 I V1: renamed from J3
- moved REF** 0.64 mm to (156.2, 109.9)
- renumbered J1 to RF1, J2 to RF2
Routing:
- net Net-(J1-Pad1): track 13.5 -> 17.4 mm
- net Net-(J2-Pad1): track 13.0 -> 17.0 mm
- net GND: vias 85 -> 83
Other:
- board outline added: 60.3 x 31.8 mm
- board text added: "2019"

Commit message: update-version
Parts:
- renumbered REF** to GND
Connections:
- GND pad 1: (no net) -> GND
Routing:
- net GND: track 20.6 -> 34.1 mm
Changed lines of the file:
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@@
     (thickness 1.6)
     (drawings 5)
-    (tracks 113)
+    (tracks 117)
     (zones 0)
     (modules 12)
@@
       (drillshape 0)
       (scaleselection 1)
-      (outputdirectory "gbr/"))
+      (outputdirectory "./"))
   )
   (net 0 "")
@@
     (descr "Through hole straight socket strip, 1x01, 1.27mm pitch, single row (from Kicad 4.0.7), script generated")
     (tags "Through hole socket strip THT 1x01 1.27mm single row")
-    (fp_text reference REF** (at 0 -2.135) (layer F.SilkS) hide
+    (fp_text reference GND (at 0 -2.135) (layer F.SilkS)
       (effects (font (size 1 1) (thickness 0.15)))
     )
@@
       (effects (font (size 0.76 0.76) (thickness 0.11)))
     )
-    (pad 1 thru_hole circle (at 0 0) (size 1 1) (drill 0.7) (layers *.Cu *.Mask))
+    (pad 1 thru_hole circle (at 0 0) (size 1 1) (drill 0.7) (layers *.Cu *.Mask)
+      (net 1 GND))
     (model ${KISYS3DMOD}/Connector_PinSocket_1.27mm.3dshapes/PinSocket_1x01_P1.27mm_Vertical.wrl
       (at (xyz 0 0 0))
@@
     (descr "Through hole straight socket strip, 1x01, 1.27mm pitch, single row (from Kicad 4.0.7), script generated")
     (tags "Through hole socket strip THT 1x01 1.27mm single row")
-    (fp_text reference REF** (at 0 -2.135) (layer F.SilkS) hide
+    (fp_text reference GND (at 0 -2.135) (layer F.SilkS)
       (effects (font (size 1 1) (thickness 0.15)))
     )
@@
   (via (at 123.19 116.84) (size 0.8) (drill 0.4) (layers F.Cu B.Cu) (net 1))
   (via (at 125.73 116.84) (size 0.8) (drill 0.4) (layers F.Cu B.Cu) (net 1))
+  (segment (start 142.24 110.49) (end 144.78 113.03) (width 0.4) (layer F.Cu) (net 1))
+  (segment (start 144.78 113.03) (end 144.78 116.205) (width 0.4) (layer F.Cu) (net 1))
+  (segment (start 121.92 110.49) (end 119.38 113.03) (width 0.4) (layer F.Cu) (net 1))
+  (segment (start 119.38 113.03) (end 119.38 116.205) (width 0.4) (layer F.Cu) (net 1))
   (segment (start 117.344999 118.240001) (end 116.84 118.745) (width 0.4) (layer F.Cu) (net 2))
   (segment (start 124.46 118.11) (end 124.590001 118.240001) (width 0.4) (layer F.Cu) (net 2))
